File: timer.sch (KiCad schematic (older format))
At the start: 29 parts, among them P1 CONN_SPI, P10 TP_DB7, P11 TP_PWR_CTRL, P12 TP_ROTA, P13 TP_ROTB, P2 PWR_IN, P3 CONN_ARDUINO_PRO_MINI_1_12, P4 CONN_ARDUINO_PRO_MINI_13_24, P5 CONN_HD44780, P6 CONN_LOAD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

Commit message: Removed bug notification from schematics...
...it is already fixed.
Other:
- note removed: "BUG: PD1 is pin 1, \n PD0 is pin 2"
Changed lines of the file:
@@
 Wire Notes Line
 	10000 2150 8900 2150
-Text Notes 5575 800  0    60   ~ 0
-BUG: PD1 is pin 1, \n         PD0 is pin 2
 $Comp
 L CONN_ARDUINO_PRO_MINI_1_12 P3
